Commit message: modificato urdf simplecar

File: f10_racecar/simplecar.urdf (robot description, URDF)
Before this commit: robot simplecar, 7 links, 6 joints
Links:
- added link camera_link, mass 0.01
- added link laser, mass 0.130; collision box size=0.1 0.1 0.1; visual mesh filename=meshes/hokuyo.obj
- added link zed_camera_link, mass 0.1; collision box size=0.033 0.175 0.030; visual box size=0.033 0.175 0.030
- added link zed_camera_right_link, mass 0.01
Joints:
- added joint hokuyo_joint: type fixed, parent base_link, child laser, origin xyz=0.1 0.0 0.075 rpy=0 0 0, axis 0 0 1
- added joint zed_camera_joint: type fixed, parent base_link, child zed_camera_link, origin xyz=0.25 0 0.04 rpy=0 0 0, axis 0 0 1
- added joint zed_camera_left_joint: type fixed, parent zed_camera_link, child camera_link, origin xyz=0 0.06 0 rpy=0 0 0, axis 0 0 1
- added joint zed_camera_right_joint: type fixed, parent zed_camera_link, child zed_camera_right_link, origin xyz=0 -0.06 0 rpy=0 0 0, axis 0 0 1

Commit message: modificato train con Adam e possibilità nuovo ambiente con cubi
modificata anche la zed in altezza altrimenti vedeva la ruota

File: f10_racecar/simplecar.urdf (robot description, URDF)
Before this commit: robot simplecar, 11 links, 10 joints
Joints:
- joint zed_camera_joint: origin xyz=0.25 0 0.04 rpy=0 0 0 -> xyz=0.35 0 0.1 rpy=0 0 0

Commit message: p control and bird_eye (da modificare)

File: f10_racecar/simplecar.urdf (robot description, URDF)
Before this commit: robot simplecar, 11 links, 10 joints
Joints:
- joint zed_camera_joint: origin xyz=0.35 0 0.1 rpy=0 0 0 -> xyz=0.35 0 0.8 rpy=0 0 0

Commit message: bird eye with edges

File: f10_racecar/simplecar.urdf (robot description, URDF)
Before this commit: robot simplecar, 11 links, 10 joints
Joints:
- joint zed_camera_joint: origin xyz=0.35 0 0.8 rpy=0 0 0 -> xyz=0.32 0 0.6 rpy=0 0 0

Commit message: ripreso vecchio modello di rete (funziona)

File: f10_racecar/simplecar.urdf (robot description, URDF)
Before this commit: robot simplecar, 11 links, 10 joints
Joints:
- joint zed_camera_joint: origin xyz=0.32 0 0.6 rpy=0 0 0 -> xyz=1 0 1 rpy=0 89 0

Commit message: adjust bird eye and start hyperparameter tuning with optuna

File: f10_racecar/simplecar.urdf (robot description, URDF)
Before this commit: robot simplecar, 11 links, 10 joints
Joints:
- joint zed_camera_joint: origin xyz=1 0 1 rpy=0 89 0 -> xyz=0.35 0 0.6 rpy=0 0 0
